File: PCB/KiCad 9 Files/Xii-Flex Ultra/Xii-Flex Ultra.kicad_pcb (KiCad board)
At the start: 2 copper layers, 47 x 56.4 mm, 3 parts, among them J1 Conn_01x50_Pin

Commit message: Add files via upload
Parts:
- moved J1 2.22 mm to (132.3, 136.4)
Routing:
- net GND: track 328.1 -> 307.4 mm
- net Net-(J1-Pin_7): track 27.3 -> 23.7 mm
- net Net-(GPIO1-Pin_1): track 37.5 -> 33.9 mm
- net Net-(J1-Pin_8): track 27.3 -> 23.7 mm
- net Net-(GCC1-Pin_1): track 37.7 -> 34.1 mm
- net Net-(J1-Pin_41): track 55.1 -> 51.5 mm
- net Net-(J1-Pin_30): track 56.8 -> 53.2 mm
- net Net-(J1-Pin_13): track 41.5 -> 37.9 mm
- net Net-(J1-Pin_9): track 27.5 -> 23.9 mm
- net Net-(J1-Pin_6): track 27.3 -> 23.7 mm
- net Net-(J1-Pin_5): track 27.3 -> 23.7 mm
- net Net-(J1-Pin_10): track 27.8 -> 24.2 mm
- net Net-(J1-Pin_46): track 57.4 -> 53.8 mm
- net Net-(J1-Pin_45): track 56.9 -> 53.3 mm
- net Net-(J1-Pin_43): track 56.1 -> 52.5 mm
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Other:
- board size 47 x 56.4 mm -> 47 x 54.1 mm
